Commit message: Comit code brisé, mais pas pire

File: urdf/3dof.urdf (robot description, URDF)
Before this commit: robot universal_robot, 9 links, 8 joints
Links:
- removed link wrist_1_link
- removed link wrist_2_link
- removed link wrist_3_link
Joints:
- removed joint wrist_1_joint
- removed joint wrist_2_joint
- removed joint wrist_3_joint
- joint ee_fixed_joint: parent wrist_3_link -> forearm_link

Commit message: Ça marcheok, mais pas assez fort

File: urdf/3dof.urdf (robot description, URDF)
Before this commit: robot universal_robot, 6 links, 5 joints
Joints:
- joint ee_fixed_joint: origin xyz=0.0 0.0823 0.0 rpy=0.0 0.0 1.57079632679 -> xyz=0.0 0.0 0.39225 rpy=0.0 0.0 0.0

File: urdf/ur5.urdf (robot description, URDF)
Before this commit: robot universal_robot, 9 links, 8 joints
Joints:
- joint wrist_1_joint: origin xyz=0.0 0.0 0.39225 rpy=0.0 1.57079632679 0.0 -> xyz=0.0 0.0 0.5 rpy=0.0 1.57079632679 0.0

Commit message: cest rigolo

File: urdf/3dof.urdf (robot description, URDF)
Before this commit: robot universal_robot, 6 links, 5 joints
Joints:
- joint elbow_joint: limit lower=-3.14159265359 upper=3.14159265359 effort=150.0 velocity=3.15 -> lower=-3.14159265359 upper=3.14159265359 effort=1000.0 velocity=3.15
- joint shoulder_lift_joint: limit lower=-6.28318530718 upper=6.28318530718 effort=150.0 velocity=3.15 -> lower=-6.28318530718 upper=6.28318530718 effort=1000.0 velocity=3.15
- joint shoulder_pan_joint: limit lower=-6.28318530718 upper=6.28318530718 effort=150.0 velocity=3.15 -> lower=-6.28318530718 upper=6.28318530718 effort=1000.0 velocity=3.15

File: urdf/ur5.urdf (robot description, URDF)
Before this commit: robot universal_robot, 9 links, 8 joints
Joints:
- joint wrist_1_joint: origin xyz=0.0 0.0 0.5 rpy=0.0 1.57079632679 0.0 -> xyz=0.0 0.0 0.39225 rpy=0.0 1.57079632679 0.0
